File: Hardware/2FA Key.kicad_sch (KiCad schematic)
At the start: 22 parts, among them J1 USB_A_PCB_Edge_receptacle, J2 Conn_ARM_SWD_TagConnect_TC203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, SW1 Push Button, U1 USBLC6-2SC6, U2 ATECC608B-SSHDA, U3 AP2112K‑3.3, U4 STM32L432KCU6

Commit message: Reorganize repo and rewrite README; add Ed25519 and compliance/programmable content
Move SSH guide to Guides/ and FIDO/RoHS docs to Compliance/; add Programmable/ (HID Injection, Mouse Jiggler, hardware, case), 3D Printable/, BOM datasheets, renders. Rewrite README around 2FAK V1C and Programmable 2FAK with Getting Started, Compliance, Resources, Credits. Resident firmware: Ed25519 (ed25519-sk) via TweetNaCl + provisioning docs. Ignore editor .history/.
Parts:
- J2: value Conn_ARM_SWD_TagConnect_TC2030-NL -> SOIC-8 Test Clamp
Changed lines of the file:
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@@
 		(title "2FAK")
 		(date "2026-09-22")
-		(rev "V1C")
+		(rev "V1CR1")
 		(company "muru.global")
 		(comment 1 "Design by Papathought")
@@
 			)
 		)
-		(property "Value" "Conn_ARM_SWD_TagConnect_TC2030-NL"
+		(property "Value" "SOIC-8 Test Clamp"
 			(at 240.03 100.3299 0)
 			(show_name no)

Commit message: Small update
Parts:
- renumbered C7 to C3, C6 to C4, C8 to C6, C3 to C7, C4 to C8, R3 to R1, R4 to R3, R5 to R4, R1 to R5, U4 to U1, U3 to U2, U2 to U3, U1 to U4
